File: botao_colibri/colibri_pcb_qfn.kicad_sch (KiCad schematic)
At the start: 6 parts, among them J2 TC2030, U1 ME54BS12

Commit message: chore: Update PCB/schematic edits and project files
Marks hole positions on the board, syncs KiCad project/prl files after
enabling the colibri-v4 library, and adds the botao_colibri KiCad
project files plus recent backup snapshots.

Co-Authored-By: Claude Sonnet 5 <noreply@anthropic.com>
Parts:
- R2, R3: value R_Small -> 4.7kR
Connections:
- net BUZZER_PWM_N renamed P2_SQUARE_WAVE
- net BUZZER_PWM_P renamed P2_SENSE
- net PROX_INT : no longer names the net of U1.7 (P1.02/NFC1)
Other:
- moved on the sheet: R2
Changed lines of the file:
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@@
 	(wire
 		(pts
-			(xy 199.39 81.28) (xy 199.39 88.9)
+			(xy 119.38 85.09) (xy 127 85.09)
+		)
+		(stroke
+			(width 0)
+			(type default)
+		)
+	)
+	(wire
+		(pts
+			(xy 190.5 81.28) (xy 190.5 88.9)
+		)
+		(stroke
+			(width 0)
+			(type default)
+		)
+	)
+	(wire
+		(pts
+			(xy 152.4 76.2) (xy 158.75 76.2)
 		)
 		(stroke
@@
 	(wire
 		(pts
-			(xy 152.4 76.2) (xy 158.75 76.2)
-		)
-		(stroke
-			(width 0)
-			(type default)
-		)
-	)
-	(wire
-		(pts
 			(xy 152.4 68.58) (xy 173.99 68.58)
 		)
@@
 	(wire
 		(pts
-			(xy 199.39 88.9) (xy 213.36 88.9)
+			(xy 190.5 88.9) (xy 213.36 88.9)
 		)
 		(stroke
@@
 	(wire
 		(pts
-			(xy 119.38 87.63) (xy 127 87.63)
-		)
-		(stroke
-			(width 0)
-			(type default)
-		)
-	)
-	(wire
-		(pts
-			(xy 199.39 69.85) (xy 199.39 76.2)
-		)
-		(stroke
-			(width 0)
-			(type default)
-		)
-	)
-	(wire
-		(pts
 			(xy 209.55 113.03) (xy 214.63 113.03)
 		)
@@
 	(wire
 		(pts
-			(xy 119.38 85.09) (xy 127 85.09)
+			(xy 190.5 68.58) (xy 190.5 76.2)
 		)
 		(stroke
@@
 		)
 	)
+	(global_label "P2_SENSE"
+		(shape input)
+		(at 119.38 85.09 180)
+		(fields_autoplaced yes)
+		(effects
+			(font
+				(size 1.27 1.27)
+			)
+			(justify right)
+		)
+		(property "Intersheetrefs" "${INTERSHEET_REFS}"
+			(at 106.9002 85.09 0)
+			(hide yes)
+			(show_name no)
+			(do_not_autoplace no)
+			(effects
+				(font
+					(size 1.27 1.27)
+				)
+				(justify right)
+			)
+		)
+	)
 	(global_label "SWDIO"
 		(shape input)
@@
 		)
 	)
+	(global_label "P2_SQUARE_WAVE"
+		(shape input)
+		(at 119.38 82.55 180)
+		(fields_autoplaced yes)
+		(effects
+			(font
+				(size 1.27 1.27)
+			)
+			(justify right)
+		)
+		(property "Intersheetrefs" "${INTERSHEET_REFS}"
+			(at 99.8244 82.55 0)
+			(hide yes)
+			(show_name no)
+			(do_not_autoplace no)
+			(effects
+				(font
+					(size 1.27 1.27)
+				)
+				(justify right)
+			)
+		)
+	)
 	(global_label "I2S_WS"
 		(shape input)
@@
 		)
 	)
-	(global_label "BUZZER_PWM_N"
-		(shape input)
-		(at 119.38 82.55 180)
+	(global_label "I2S_SD"
+		(shape input)
+		(at 119.38 80.01 180)
 		(fields_autoplaced yes)
 		(effects
@@
 		)
 		(property "Intersheetrefs" "${INTERSHEET_REFS}"
-			(at 101.5178 82.55 0)
+			(at 109.9239 80.01 0)
 			(hide yes)
 			(show_name no)
@@
 		)
 	)
-	(global_label "I2S_SD"
-		(shape input)
-		(at 119.38 80.01 180)
+	(global_label "LED_R"
+		(shape input)
+		(at 119.38 90.17 180)
 		(fields_autoplaced yes)
 		(effects
@@
 		)
 		(property "Intersheetrefs" "${INTERSHEET_REFS}"
-			(at 109.9239 80.01 0)
-			(hide yes)
-			(show_name no)
-			(do_not_autoplace no)
-			(effects
-				(font
-					(size 1.27 1.27)
-				)
-				(justify right)
-			)
-		)
-	)
-	(global_label "BUZZER_PWM_P"
-		(shape input)
-		(at 119.38 85.09 180)
-		(fields_autoplaced yes)
-		(effects
-			(font
-				(size 1.27 1.27)
-			)
-			(justify right)
-		)
-		(property "Intersheetrefs" "${INTERSHEET_REFS}"
-			(at 101.5783 85.09 0)
-			(hide yes)
-			(show_name no)
-			(do_not_autoplace no)
-			(effects
-				(font
-					(size 1.27 1.27)
-				)
-				(justify right)
-			)
-		)
-	)
-	(global_label "LED_R"
-		(shape input)
-		(at 119.38 90.17 180)
-		(fields_autoplaced yes)
-		(effects
-			(font
-				(size 1.27 1.27)
-			)
-			(justify right)
-		)
-		(property "Intersheetrefs" "${INTERSHEET_REFS}"
 			(at 110.7101 90.17 0)
-			(hide yes)
-			(show_name no)
-			(do_not_autoplace no)
-			(effects
-				(font
-					(size 1.27 1.27)
-				)
-				(justify right)
-			)
-		)
-	)
-	(global_label "PROX_INT "
-		(shape input)
-		(at 119.38 87.63 180)
-		(fields_autoplaced yes)
-		(effects
-			(font
-				(size 1.27 1.27)
-			)
-			(justify right)
-		)
-		(property "Intersheetrefs" "${INTERSHEET_REFS}"
-			(at 106.4767 87.63 0)
 			(hide yes)
 			(show_name no)
@@
 	(symbol
 		(lib_id "Device:R_Small")
-		(at 199.39 78.74 180)
+		(at 190.5 78.74 180)
 		(unit 1)
 		(body_style 1)
@@
 		(dnp no)
 		(property "Reference" "R2"
-			(at 201.168 77.216 0)
+			(at 192.278 77.216 0)
 			(show_name no)
 			(do_not_autoplace no)
@@
 			)
 		)
-		(property "Value" "R_Small"
-			(at 201.93 80.0099 0)
-			(hide yes)
+		(property "Value" "4.7kR"
+			(at 193.04 80.0099 0)
 			(show_name no)
 			(do_not_autoplace no)
@@
 		)
 		(property "Footprint" "Resistor_SMD:R_0402_1005Metric_Pad0.72x0.64mm_HandSolder"
-			(at 199.39 78.74 0)
+			(at 190.5 78.74 0)
 			(hide yes)
 			(show_name no)
@@
 		)
 		(property "Datasheet" ""
-			(at 199.39 78.74 0)
+			(at 190.5 78.74 0)
 			(hide yes)
 			(show_name no)
@@
 		)
 		(property "Description" "Resistor, small symbol"
-			(at 199.39 78.74 0)
+			(at 190.5 78.74 0)
 			(hide yes)
 			(show_name no)
@@
 			)
 		)
-		(property "Value" "R_Small"
+		(property "Value" "4.7kR"
 			(at 207.01 80.0099 0)
-			(hide yes)
 			(show_name no)
 			(do_not_autoplace no)
@@
 	(symbol
 		(lib_id "power:VDD")
-		(at 199.39 69.85 0)
+		(at 190.5 68.58 0)
 		(unit 1)
 		(body_style 1)
@@
 		(fields_autoplaced yes)
 		(property "Reference" "#PWR027"
-			(at 199.39 73.66 0)
+			(at 190.5 72.39 0)
 			(hide yes)
 			(show_name no)
@@
 		)
 		(property "Value" "VDD"
-			(at 199.39 64.77 0)
+			(at 190.5 63.5 0)
 			(show_name no)
 			(do_not_autoplace no)
@@
 		)
 		(property "Footprint" ""
-			(at 199.39 69.85 0)
+			(at 190.5 68.58 0)
 			(hide yes)
 			(show_name no)
@@
 		)
 		(property "Datasheet" ""
-			(at 199.39 69.85 0)
+			(at 190.5 68.58 0)
 			(hide yes)
 			(show_name no)
@@
 		)
 		(property "Description" "Power symbol creates a global label with name \"VDD\""
-			(at 199.39 69.85 0)
-			(hide yes)
-			(show_name no)
+			(at 190.5 68.58 0)
+			(hide yes)
+			(show_name no)
