File: botao_colibri/colibri_pcb_qfn.kicad_sch (KiCad schematic)
At the start: 6 parts, among them J2 TC2030, U1 ME54BS12

Commit message: Posicionamento inicial dos componentes na pcb e alguns ajustes no esquemático
Connections:
- net VDD: now also R2.2
- no-connect marks 16 -> 19
Changed lines of the file:
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@@
+	)
+	(no_connect
+		(at 127 87.63)
 	)
 	(no_connect
@@
 	)
 	(no_connect
+		(at 152.4 86.36)
+	)
+	(no_connect
 		(at 152.4 91.44)
 	)
@@
 	)
 	(no_connect
+		(at 152.4 111.76)
+	)
+	(no_connect
 		(at 127 105.41)
 	)
@@
 	(wire
 		(pts
-			(xy 158.75 86.36) (xy 152.4 86.36)
-		)
-		(stroke
-			(width 0)
-			(type default)
-		)
-	)
-	(wire
-		(pts
 			(xy 119.38 80.01) (xy 127 80.01)
 		)
@@
 		)
 		(stroke
+			(width 0)
+			(type default)
+		)
+	)
+	(wire
+		(pts
+			(xy 190.5 68.58) (xy 190.5 76.2)
+		)
+		(stroke
