File: botao_colibri/power_management.kicad_sch (KiCad schematic)
At the start: 24 parts, among them J1 USB4970-00-A_REVA, J3 Conn_01x02, SW1 B3F-3122, U4 NPM1300-QEAA-R7

Commit message: Avanço nos posicionamentos
Changed lines of the file:
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@@
 	(wire
 		(pts
-			(xy 87.63 80.01) (xy 91.44 80.01)
+			(xy 87.63 81.28) (xy 88.9 81.28)
 		)
 		(stroke
@@
 	(wire
 		(pts
+			(xy 88.9 81.28) (xy 88.9 80.01)
+		)
+		(stroke
+			(width 0)
+			(type default)
+		)
+	)
+	(wire
+		(pts
 			(xy 115.57 39.37) (xy 118.11 39.37)
 		)
@@
 		(pts
 			(xy 161.29 80.01) (xy 157.48 80.01)
+		)
+		(stroke
+			(width 0)
+			(type default)
+		)
+	)
+	(wire
+		(pts
+			(xy 88.9 80.01) (xy 91.44 80.01)
 		)
 		(stroke
@@
 	(global_label "PVDD"
 		(shape input)
-		(at 87.63 80.01 180)
+		(at 87.63 81.28 180)
 		(fields_autoplaced yes)
 		(effects
@@
 		)
 		(property "Intersheetrefs" "${INTERSHEET_REFS}"
-			(at 79.7462 80.01 0)
+			(at 79.7462 81.28 0)
 			(hide yes)
 			(show_name no)
